File: drone-esc-module.kicad_pcb (KiCad board)
At the start: 2 copper layers, 18.2 x 18.2 mm, 1 part

Commit message: done with schematic fr
Parts:
- added C10: 10u, Capacitor_SMD:C_0805_2012Metric, F.Cu at (161.8, 86.7)
- added C25: 100n, Capacitor_SMD:C_0201_0603Metric, F.Cu at (157.8, 98.8)
- added C26: 100n, Capacitor_SMD:C_0201_0603Metric, F.Cu at (157.8, 100.5)
- added C28: 100n, Capacitor_SMD:C_0201_0603Metric, F.Cu at (149.4, 108.8)
- added C29: 100n, Capacitor_SMD:C_0201_0603Metric, F.Cu at (161.6, 108.8)
- added C3: 1u, Capacitor_SMD:C_0201_0603Metric, F.Cu at (157.8, 95.3)
- added C30: 100n, Capacitor_SMD:C_0201_0603Metric, F.Cu at (137.3, 108.8)
- added C4: 2u2, Capacitor_SMD:C_0201_0603Metric, F.Cu at (157.8, 97.0)
- added C43: 100n, Capacitor_SMD:C_0201_0603Metric, F.Cu at (149.4, 110.5)
- added C44: 100n, Capacitor_SMD:C_0201_0603Metric, F.Cu at (161.6, 110.5)
- added C45: 100n, Capacitor_SMD:C_0201_0603Metric, F.Cu at (160.2, 95.3)
- added C46: 100n, Capacitor_SMD:C_0201_0603Metric, F.Cu at (137.3, 110.5)
- added C8: 10u, Capacitor_SMD:C_0805_2012Metric, F.Cu at (161.8, 80.7)
- added C9: 10u, Capacitor_SMD:C_0805_2012Metric, F.Cu at (161.8, 83.7)
- added D2: HSMD-C170, LED_SMD:LED_0805_2012Metric, F.Cu at (144.9, 101.2)
- added D4: HSMG-C170, LED_SMD:LED_0805_2012Metric, F.Cu at (144.9, 104.2)
- added FB1: BLM03HD331SN1D, Resistor_SMD:R_0201_0603Metric, F.Cu at (160.2, 97.0)
- added Q10: IRLHS6242, IRLHS6242TRPBF:IRL100HS121-V, F.Cu at (165.4, 113.6)
- added Q11: IRLHS6242, IRLHS6242TRPBF:IRL100HS121-V, F.Cu at (141.1, 109.8)
- added Q12: IRLHS6242, IRLHS6242TRPBF:IRL100HS121-V, F.Cu at (141.1, 113.6)
- added Q7: IRLHS6242, IRLHS6242TRPBF:IRL100HS121-V, F.Cu at (153.3, 109.8)
- added Q8: IRLHS6242, IRLHS6242TRPBF:IRL100HS121-V, F.Cu at (153.3, 113.6)
- added Q9: IRLHS6242, IRLHS6242TRPBF:IRL100HS121-V, F.Cu at (165.4, 109.8)
- added R11: 100k, Resistor_SMD:R_0201_0603Metric, F.Cu at (149.4, 112.3)
- added R12: 100k, Resistor_SMD:R_0201_0603Metric, F.Cu at (161.6, 112.3)
- added R13: 100k, Resistor_SMD:R_0201_0603Metric, F.Cu at (137.3, 112.3)
- added R26: 15R, Resistor_SMD:R_0201_0603Metric, F.Cu at (149.4, 114.0)
- added R27: 4.7k, Resistor_SMD:R_0201_0603Metric, F.Cu at (149.4, 115.8)
- added R28: 10k, Resistor_SMD:R_0201_0603Metric, F.Cu at (149.4, 117.5)
- added R29: 1k, Resistor_SMD:R_0201_0603Metric, F.Cu at (149.4, 119.3)
- added R30: 4.7k, Resistor_SMD:R_0201_0603Metric, F.Cu at (161.6, 114.0)
- added R31: 10k, Resistor_SMD:R_0201_0603Metric, F.Cu at (161.6, 115.8)
- added R32: 1k, Resistor_SMD:R_0201_0603Metric, F.Cu at (161.6, 117.5)
- added R33: 15R, Resistor_SMD:R_0201_0603Metric, F.Cu at (161.6, 119.3)
- added R34: 4.7k, Resistor_SMD:R_0201_0603Metric, F.Cu at (137.3, 114.0)
- added R35: 10k, Resistor_SMD:R_0201_0603Metric, F.Cu at (137.3, 115.8)
- added R36: 1k, Resistor_SMD:R_0201_0603Metric, F.Cu at (137.3, 117.5)
- added R37: 15R, Resistor_SMD:R_0201_0603Metric, F.Cu at (137.3, 119.3)
- added R47: 10k, Resistor_SMD:R_0201_0603Metric, F.Cu at (162.7, 97.0)
- added R5: 360, Resistor_SMD:R_0201_0603Metric, F.Cu at (160.2, 98.8)
- added R54: 15R, Resistor_SMD:R_0201_0603Metric, F.Cu at (149.4, 121.0)
- added R55: 15R, Resistor_SMD:R_0201_0603Metric, F.Cu at (161.6, 121.0)
- added R56: 15R, Resistor_SMD:R_0201_0603Metric, F.Cu at (137.3, 121.0)
- added R6: 10k, Resistor_SMD:R_0201_0603Metric, F.Cu at (160.2, 100.5)
- added R7: 220R, Resistor_SMD:R_0201_0603Metric, F.Cu at (162.7, 95.3)
- added R91: 360, Resistor_SMD:R_0201_0603Metric, F.Cu at (162.7, 98.8)
- added TP16: 3V3, TestPoint:TestPoint_Pad_D1.0mm, F.Cu at (158.1, 89.8)
- added TP19: BOOT0, TestPoint:TestPoint_Pad_D1.0mm, F.Cu at (158.1, 92.9)
- added TP2: SWCLK, TestPoint:TestPoint_Pad_D1.0mm, F.Cu at (158.1, 80.7)
- added TP25: GH, TestPoint:TestPoint_Pad_D1.0mm, F.Cu at (156.8, 109.4)
- added TP26: GH, TestPoint:TestPoint_Pad_D1.0mm, F.Cu at (169.0, 109.4)
- added TP27: GH, TestPoint:TestPoint_Pad_D1.0mm, F.Cu at (144.7, 109.4)
- added TP3: NRST, TestPoint:TestPoint_Pad_D1.0mm, F.Cu at (158.1, 83.7)
- added TP37: GL, TestPoint:TestPoint_Pad_D1.0mm, F.Cu at (156.8, 112.5)
- added TP38: GL, TestPoint:TestPoint_Pad_D1.0mm, F.Cu at (169.0, 112.5)
- added TP39: GL, TestPoint:TestPoint_Pad_D1.0mm, F.Cu at (144.7, 112.5)
- added TP9: SWDIO, TestPoint:TestPoint_Pad_D1.0mm, F.Cu at (158.1, 86.8)
- added U10: DGD05473FNQ-7, Package_DFN_QFN:DFN-10-1EP_3x3mm_P0.5mm_EP1.7x2.5mm, F.Cu at (165.8, 117.7)
- added U11: DGD05473FNQ-7, Package_DFN_QFN:DFN-10-1EP_3x3mm_P0.5mm_EP1.7x2.5mm, F.Cu at (141.5, 117.7)
- added U3: TLV76733DRVR, Package_SON:WSON-6-1EP_2x2mm_P0.65mm_EP1x1.6mm_ThermalVias, F.Cu at (149.0, 101.5)
- added U5: AT32F421G8U7, Package_DFN_QFN:QFN-28-1EP_4x4mm_P0.45mm_EP2.4x2.4mm, F.Cu at (139.6, 102.8)
- added U9: DGD05473FNQ-7, Package_DFN_QFN:DFN-10-1EP_3x3mm_P0.5mm_EP1.7x2.5mm, F.Cu at (153.7, 117.7)
- moved U1 32.7 mm to (155.8, 98.9)
Connections:
- U1 pad 2: +BATT -> GND
- U1 pad 4: /MOTORA -> +BATT
- U1 pad 5: /MOTORB -> /MOTORA
- U1 pad 6: /MOTORC -> /MOTORB
- U1 pad 7: GND -> /MOTORC
Other:
- board size 18.2 x 18.2 mm -> 18.5 x 18.5 mm
