File: drone-esc-module.kicad_sch (KiCad schematic)
At the start: 24 parts, among them U3 TLV76733DRVR, U5 AT32F421G8U7

Commit message: finish schematic + footprints
Connections:
- net +5V: now also U1.3 (+5V); no longer U1. (DSHOT)
- net +BATT: now also U1.2 (+BATT); no longer U1. (DSHOT)
- net DSHOT: now also U1.1 (DSHOT); no longer U1. (DSHOT)
- net GND: now also U1.7 (GND)
- net MOTORA: now also U1.4 (MOTORA); no longer U1. (DSHOT)
- net MOTORB: now also U1.5 (MOTORB); no longer U1. (DSHOT)
- net MOTORC: now also U1.6 (MOTORC); no longer U1. (DSHOT)

Commit message: done with schematic fr
Connections:
- net +BATT: now also U1.4 (+BATT); no longer U1.2 (+BATT)
- net GND: now also U1.2 (GND); no longer U1.7 (GND)
- net MOTORA: now also U1.5 (MOTORA); no longer U1.4 (MOTORA)
- net MOTORB: now also U1.6 (MOTORB); no longer U1.5 (MOTORB)
- net MOTORC: now also U1.7 (MOTORC); no longer U1.6 (MOTORC)
Other:
- moved on the sheet: U1
Changed lines of the file:
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@@
 	(wire
 		(pts
+			(xy 243.84 25.4) (xy 243.84 38.1)
+		)
+		(stroke
+			(width 0)
+			(type default)
+		)
+	)
+	(wire
+		(pts
 			(xy 95.25 25.4) (xy 95.25 27.94)
 		)
@@
 	(wire
 		(pts
-			(xy 181.61 128.27) (xy 186.69 128.27)
+			(xy 255.27 26.67) (xy 255.27 25.4)
 		)
 		(stroke
@@
 	(wire
 		(pts
-			(xy 181.61 124.46) (xy 186.69 124.46)
+			(xy 181.61 128.27) (xy 186.69 128.27)
 		)
 		(stroke
@@
 	(wire
 		(pts
-			(xy 73.66 123.19) (xy 69.85 123.19)
+			(xy 181.61 124.46) (xy 186.69 124.46)
 		)
 		(stroke
@@
 	(wire
 		(pts
-			(xy 73.66 127) (xy 69.85 127)
+			(xy 73.66 123.19) (xy 69.85 123.19)
 		)
 		(stroke
@@
 	(wire
 		(pts
-			(xy 148.59 105.41) (xy 143.51 105.41)
+			(xy 73.66 127) (xy 69.85 127)
 		)
 		(stroke
@@
 	(wire
 		(pts
-			(xy 67.31 172.72) (xy 67.31 170.18)
+			(xy 148.59 105.41) (xy 143.51 105.41)
 		)
 		(stroke
@@
 	(wire
 		(pts
-			(xy 148.59 171.45) (xy 148.59 172.72)
+			(xy 67.31 172.72) (xy 67.31 170.18)
 		)
 		(stroke
@@
 	(wire
 		(pts
-			(xy 259.08 59.69) (xy 255.27 59.69)
+			(xy 148.59 171.45) (xy 148.59 172.72)
 		)
 		(stroke
@@
 	(wire
 		(pts
+			(xy 255.27 25.4) (xy 243.84 25.4)
+		)
+		(stroke
+			(width 0)
+			(type default)
+		)
+	)
+	(wire
+		(pts
 			(xy 38.1 115.57) (xy 40.64 115.57)
 		)
@@
 		)
 	)
-	(label "+BATT"
-		(at 241.3 38.1 90)
-		(effects
-			(font
-				(size 1.27 1.27)
-			)
-			(justify left bottom)
-		)
-	)
 	(label "BOOT0"
 		(at 71.12 50.8 0)
@@
 	)
 	(label "+5V"
-		(at 236.22 38.1 90)
+		(at 238.76 38.1 90)
 		(effects
 			(font
@@
 	)
 	(label "DSHOT"
-		(at 247.65 38.1 90)
+		(at 250.19 38.1 90)
 		(effects
 			(font
@@
 		)
 	)
+	(label "+BATT"
+		(at 233.68 38.1 90)
+		(effects
+			(font
+				(size 1.27 1.27)
+			)
+			(justify left bottom)
+		)
+	)
 	(label "+5V"
 		(at 220.98 105.41 0)
@@
 	(symbol
 		(lib_id "power:GND")
-		(at 259.08 59.69 0)
-		(unit 1)
-		(body_style 1)
-		(exclude_from_sim no)
-		(in_bom yes)
-		(on_board yes)
-		(in_pos_files yes)
-		(dnp no)
-		(fields_autoplaced yes)
-		(property "Reference" "#PWR043"
-			(at 259.08 66.04 0)
-			(hide yes)
-			(show_name no)
-			(do_not_autoplace no)
-			(effects
-				(font
-					(size 1.27 1.27)
-				)
-			)
-		)
-		(property "Value" "GND"
-			(at 259.08 64.77 0)
-			(show_name no)
-			(do_not_autoplace no)
-			(effects
-				(font
-					(size 1.27 1.27)
-				)
-			)
-		)
-		(property "Footprint" ""
-			(at 259.08 59.69 0)
-			(hide yes)
-			(show_name no)
-			(do_not_autoplace no)
-			(effects
-				(font
-					(size 1.27 1.27)
-				)
-			)
-		)
-		(property "Datasheet" ""
-			(at 259.08 59.69 0)
-			(hide yes)
-			(show_name no)
-			(do_not_autoplace no)
-			(effects
-				(font
-					(size 1.27 1.27)
-				)
-			)
-		)
-		(property "Description" "Power symbol creates a global label with name \"GND\" , ground"
-			(at 259.08 59.69 0)
-			(hide yes)
-			(show_name no)
-			(do_not_autoplace no)
-			(effects
-				(font
-					(size 1.27 1.27)
-				)
-			)
-		)
-		(pin "1"
-		)
-		(instances
-			(project "drone-esc-module"
-				(path "/5a929d07-7698-4420-af66-dd70e0412f52"
-					(reference "#PWR043")
-					(unit 1)
-				)
-			)
-		)
-	)
-	(symbol
-		(lib_id "power:GND")
 		(at 76.2 182.88 0)
 		(unit 1)
@@
 					(unit 1)
 				)
+			)
+		)
+	)
+	(symbol
+		(lib_id "power:GND")
+		(at 255.27 26.67 0)
+		(unit 1)
+		(body_style 1)
+		(exclude_from_sim no)
+		(in_bom yes)
+		(on_board yes)
+		(in_pos_files yes)
+		(dnp no)
+		(fields_autoplaced yes)
+		(property "Reference" "#PWR043"
+			(at 255.27 33.02 0)
+			(hide yes)
+			(show_name no)
+			(do_not_autoplace no)
+			(effects
+				(font
+					(size 1.27 1.27)
+				)
+			)
+		)
+		(property "Value" "GND"
+			(at 255.27 31.75 0)
+			(show_name no)
+			(do_not_autoplace no)
+			(effects
+				(font
+					(size 1.27 1.27)
+				)
+			)
+		)
+		(property "Footprint" ""
+			(at 255.27 26.67 0)
+			(hide yes)
+			(show_name no)
+			(do_not_autoplace no)
+			(effects
+				(font
+					(size 1.27 1.27)
+				)
+			)
+		)
+		(property "Datasheet" ""
+			(at 255.27 26.67 0)
+			(hide yes)
+			(show_name no)
+			(do_not_autoplace no)
+			(effects
+				(font
+					(size 1.27 1.27)
+				)
+			)
+		)
+		(property "Description" "Power symbol creates a global label with name \"GND\" , ground"
+			(at 255.27 26.67 0)
+			(hide yes)
+			(show_name no)
+			(do_not_autoplace no)
+			(effects
+				(font
+					(size 1.27 1.27)
+				)
+			)
+		)
+		(pin "1"
+		)
+		(instances
+			(project "drone-esc-module"
+				(path "/5a929d07-7698-4420-af66-dd70e0412f52"
+					(reference "#PWR043")
+					(unit 1)
+				)
